Commit message: robo.xacro working

File: urdf/robo.xacro (robot description, xacro)
@@ -1,4 +1,12 @@
 <?xml version='1.0'?>
-<robot name="lols">
+<robot name="lols" xmlns:xacro="http://www.ros.org/wiki/xacro">
+  <xacro:property name="wheel_radius" value="0.2"/>
+  <xacro:property name="wheel_thickness" value="0.1" />
+  <xacro:property name="wheel_mass" value="0.2" />
+  <xacro:property name="chassis_length" value="1" />
+  <xacro:property name="chassis_breadth" value="0.5" />
+  <xacro:property name="chassis_height" value="0.25" />
+  <xacro:property name="chassis_mass" value="5" />
+  <xacro:include filename="$(find ohno)/urdf/materials.xacro"/>
   <gazebo>
     <static>False</static>
@@ -7,11 +15,10 @@
   <!-- Base Link -->
   <link name="base_link">
+    <pose>0 0 3 0 0 0</pose>
     <visual>
-      <material name="blue">
-        <color rgba="0 0.5 1 1"/>
-      </material>
+      <material name="white"/>
       <origin xyz="0 0 0.05" rpy="0 0 0" />
       <geometry>
-          <box size="1 0.5 0.25"/>
+          <box size="${chassis_length} ${chassis_breadth} ${chassis_height}"/>
       </geometry>
     </visual>
@@ -20,13 +27,16 @@
       <origin xyz="0 0 0.05" rpy="0 0 0" />
       <geometry>
-          <box size="1 0.5 0.25"/>
+          <box size="${chassis_length} ${chassis_breadth} ${chassis_height}"/>
       </geometry>
     </collision>
     <inertial>
-      <mass value="5"/>
+      <mass value="${chassis_mass}"/>
       <inertia ixx="0.13" ixy="0.0" ixz="0.0" iyy="0.21" iyz="0.0" izz="0.13"/>
     </inertial>
-    </link>
-    <link name="right_front">
+  </link>
+  <gazebo reference="base_link">
+    <material>Gazebo/Blue</material>
+  </gazebo>
+  <link name="right_front">
         <inertial>
             <!-- <origin xyz="0.0 0.0 0.0" rpy="0.0 0.0 0.0"/> -->
@@ -36,9 +46,7 @@
         <visual>
             <origin xyz="0.0 0.0 0.0" rpy="1.570795 0.0 0.0"/>
-            <material name="black">
-                <color rgba="0.05 0.05 0.05 1"/>
-            </material>
+            <material name="black"/>
             <geometry>
-                <cylinder length="0.1" radius="0.2"/>
+                <cylinder length="${wheel_thickness}" radius="${wheel_radius}"/>
             </geometry>
         </visual>
@@ -46,5 +54,5 @@
             <origin xyz="0.0 0.0 0.0" rpy="1.570795 0.0 0.0"/>
             <geometry>
-                <cylinder length="0.1" radius="0.2" />
+                <cylinder length="${wheel_thickness}" radius="${wheel_radius}" />
             </geometry>
         </collision>
@@ -71,5 +79,5 @@
             </material>
             <geometry>
-                <cylinder length="0.1" radius="0.2"/>
+                <cylinder length="${wheel_thickness}" radius="${wheel_radius}"/>
             </geometry>
         </visual>
@@ -77,5 +85,5 @@
             <origin xyz="0.0 0.0 0.0" rpy="1.570795 0.0 0.0"/>
             <geometry>
-                <cylinder length="0.1" radius="0.2" />
+                <cylinder length="${wheel_thickness}" radius="${wheel_radius}" />
             </geometry>
         </collision>
@@ -102,5 +110,5 @@
             </material>
             <geometry>
-                <cylinder length="0.1" radius="0.2"/>
+                <cylinder length="${wheel_thickness}" radius="${wheel_radius}"/>
             </geometry>
         </visual>
@@ -108,5 +116,5 @@
             <origin xyz="0.0 0.0 0.0" rpy="1.570795 0.0 0.0"/>
             <geometry>
-                <cylinder length="0.1" radius="0.2" />
+                <cylinder length="${wheel_thickness}" radius="${wheel_radius}" />
             </geometry>
         </collision>
@@ -133,5 +141,5 @@
             </material>
             <geometry>
-                <cylinder length="0.1" radius="0.2"/>
+                <cylinder length="${wheel_thickness}" radius="${wheel_radius}"/>
             </geometry>
         </visual>
@@ -139,5 +147,5 @@
             <origin xyz="0.0 0.0 0.0" rpy="1.570795 0.0 0.0"/>
             <geometry>
-                <cylinder length="0.1" radiu0s="0.2" />
+                <cylinder length="${wheel_thickness}" radius="${wheel_radius}" />
             </geometry>
         </collision>
@@ -152,8 +160,4 @@
         <axis xyz="0 1 0"/>
     </joint>
-  <gazebo reference="base_link">
-    <material>Gazebo/Blue</material>
-    <pose>0 0 3 0 0 0</pose>
-  </gazebo>
   <joint name="dummy_joint" type="fixed">
     <origin xyz="0.0 0.0 1" rpy="0.0 0.0 0.0"/>

Commit message: Xacro-Done

File: urdf/robo.xacro (robot description, xacro)
@@ -36,5 +36,5 @@
   </link>
   <gazebo reference="base_link">
-    <material>Gazebo/Blue</material>
+    <material>Gazebo/White</material>
   </gazebo>
   <link name="right_front">
@@ -75,7 +75,5 @@
         <visual>
             <origin xyz="0.0 0.0 0.0" rpy="1.570795 0.0 0.0"/>
-            <material name="black">
-                <color rgba="0.05 0.05 0.05 1"/>
-            </material>
+            <material name="black"/>
             <geometry>
                 <cylinder length="${wheel_thickness}" radius="${wheel_radius}"/>
@@ -106,7 +104,5 @@
         <visual>
             <origin xyz="0.0 0.0 0.0" rpy="1.570795 0.0 0.0"/>
-            <material name="black">
-                <color rgba="0.05 0.05 0.05 1"/>
-            </material>
+            <material name="black"/>
             <geometry>
                 <cylinder length="${wheel_thickness}" radius="${wheel_radius}"/>
@@ -137,7 +133,5 @@
         <visual>
             <origin xyz="0.0 0.0 0.0" rpy="1.570795 0.0 0.0"/>
-            <material name="black">
-                <color rgba="0.05 0.05 0.05 1"/>
-            </material>
+            <material name="black"/>
             <geometry>
                 <cylinder length="${wheel_thickness}" radius="${wheel_radius}"/>

Commit message: Wheels with macros

File: urdf/robo.xacro (robot description, xacro)
@@ -9,4 +9,5 @@
   <xacro:property name="chassis_mass" value="5" />
   <xacro:include filename="$(find ohno)/urdf/materials.xacro"/>
+  <xacro:include filename="$(find ohno)/urdf/wheel.xacro"/>
   <gazebo>
     <static>False</static>
@@ -38,120 +39,8 @@
     <material>Gazebo/White</material>
   </gazebo>
-  <link name="right_front">
-        <inertial>
-            <!-- <origin xyz="0.0 0.0 0.0" rpy="0.0 0.0 0.0"/> -->
-            <mass value="0.5"/>
-            <inertia ixx="0.01" ixy="0.0" ixz="0.0" iyy="0.005" iyz="0.0" izz="0.005"/>
-        </inertial>
-        <visual>
-            <origin xyz="0.0 0.0 0.0" rpy="1.570795 0.0 0.0"/>
-            <material name="black"/>
-            <geometry>
-                <cylinder length="${wheel_thickness}" radius="${wheel_radius}"/>
-            </geometry>
-        </visual>
-        <collision>
-            <origin xyz="0.0 0.0 0.0" rpy="1.570795 0.0 0.0"/>
-            <geometry>
-                <cylinder length="${wheel_thickness}" radius="${wheel_radius}" />
-            </geometry>
-        </collision>
-    </link>
-    <gazebo reference ="right_front">
-        <material>Gazebo/Black</material>
-    </gazebo>
-    <joint name="joint_right_front" type="continuous">
-        <origin xyz="0.4 -0.3 0.05" rpy="0.0 0.0 0.0"/>
-        <parent link="base_link"/>
-        <child link="right_front"/>
-        <axis xyz="0 1 0"/>
-    </joint>
-    <link name="left_front">
-        <inertial>
-            <!-- <origin xyz="0.0 0.0 0.0" rpy="0.0 0.0 0.0"/> -->
-            <mass value="0.5"/>
-            <inertia ixx="0.01" ixy="0.0" ixz="0.0" iyy="0.005" iyz="0.0" izz="0.005"/>
-        </inertial>
-        <visual>
-            <origin xyz="0.0 0.0 0.0" rpy="1.570795 0.0 0.0"/>
-            <material name="black"/>
-            <geometry>
-                <cylinder length="${wheel_thickness}" radius="${wheel_radius}"/>
-            </geometry>
-        </visual>
-        <collision>
-            <origin xyz="0.0 0.0 0.0" rpy="1.570795 0.0 0.0"/>
-            <geometry>
-                <cylinder length="${wheel_thickness}" radius="${wheel_radius}" />
-            </geometry>
-        </collision>
-    </link>
-    <gazebo reference ="left_front">
-        <material>Gazebo/Black</material>
-    </gazebo>
-    <joint name="joint_left_front" type="continuous">
-        <origin xyz="0.4 0.3 0.05" rpy="0.0 0.0 0.0"/>
-        <parent link="base_link"/>
-        <child link="left_front"/>
-        <axis xyz="0 1 0"/>
-    </joint>
-    <link name="right_back">
-        <inertial>
-            <!-- <origin xyz="0.0 0.0 0.0" rpy="0.0 0.0 0.0"/> -->
-            <mass value="0.5"/>
-            <inertia ixx="0.01" ixy="0.0" ixz="0.0" iyy="0.005" iyz="0.0" izz="0.005"/>
-        </inertial>
-        <visual>
-            <origin xyz="0.0 0.0 0.0" rpy="1.570795 0.0 0.0"/>
-            <material name="black"/>
-            <geometry>
-                <cylinder length="${wheel_thickness}" radius="${wheel_radius}"/>
-            </geometry>
-        </visual>
-        <collision>
-            <origin xyz="0.0 0.0 0.0" rpy="1.570795 0.0 0.0"/>
-            <geometry>
-                <cylinder length="${wheel_thickness}" radius="${wheel_radius}" />
-            </geometry>
-        </collision>
-    </link>
-    <gazebo reference ="right_back">
-        <material>Gazebo/Black</material>
-    </gazebo>
-    <joint name="joint_right_back" type="continuous">
-        <origin xyz="-0.4 -0.3 0.05" rpy="0.0 0.0 0.0"/>
-        <parent link="base_link"/>
-        <child link="right_back"/>
-        <axis xyz="0 1 0"/>
-    </joint>
-    <link name="left_back">
-        <inertial>
-            <!-- <origin xyz="0.0 0.0 0.0" rpy="0.0 0.0 0.0"/> -->
-            <mass value="0.5"/>
-            <inertia ixx="0.01" ixy="0.0" ixz="0.0" iyy="0.005" iyz="0.0" izz="0.005"/>
-        </inertial>
-        <visual>
-            <origin xyz="0.0 0.0 0.0" rpy="1.570795 0.0 0.0"/>
-            <material name="black"/>
-            <geometry>
-                <cylinder length="${wheel_thickness}" radius="${wheel_radius}"/>
-            </geometry>
-        </visual>
-        <collision>
-            <origin xyz="0.0 0.0 0.0" rpy="1.570795 0.0 0.0"/>
-            <geometry>
-                <cylinder length="${wheel_thickness}" radius="${wheel_radius}" />
-            </geometry>
-        </collision>
-    </link>
-    <gazebo reference ="left_back">
-        <material>Gazebo/Black</material>
-    </gazebo>
-    <joint name="joint_left_back" type="continuous">
-        <origin xyz="-0.4 0.3 0.05" rpy="0.0 0.0 0.0"/>
-        <parent link="base_link"/>
-        <child link="left_back"/>
-        <axis xyz="0 1 0"/>
-    </joint>
+  <xacro:define_wheel name_a="front_right" name_b="front_right_joint"  rad="${wheel_radius}" thicc="${wheel_thickness}"  origin_xyz="0.4 -0.3 0.05"/>
+  <xacro:define_wheel name_a="front_left" name_b="front_left_joint" rad="${wheel_radius}" thicc="${wheel_thickness}" origin_xyz="0.4 0.3 0.05"/>
+  <xacro:define_wheel name_a="back_right" name_b="back_right_joint" rad="${wheel_radius}" thicc="${wheel_thickness}" origin_xyz="-0.4 -0.3 0.05"/>
+  <xacro:define_wheel name_a="back_left" name_b="back_left_joint" rad="${wheel_radius}" thicc="${wheel_thickness}" origin_xyz="-0.4 0.3 0.05"/>
   <joint name="dummy_joint" type="fixed">
     <origin xyz="0.0 0.0 1" rpy="0.0 0.0 0.0"/>

Commit message: Wheels go into ground Link pls check @leander

File: urdf/robo.xacro (robot description, xacro)
@@ -10,4 +10,5 @@
   <xacro:include filename="$(find ohno)/urdf/materials.xacro"/>
   <xacro:include filename="$(find ohno)/urdf/wheel.xacro"/>
+  <!-- <xacro:include filename="$(find ohno)/urdf/robo.gazebo"/> -->
   <gazebo>
     <static>False</static>
@@ -25,5 +26,5 @@
     </visual>
     <!-- Base collision, mass and inertia -->
-    <collision>
+    <collision>z
       <origin xyz="0 0 0.05" rpy="0 0 0" />
       <geometry>
@@ -36,11 +37,23 @@
     </inertial>
   </link>
-  <gazebo reference="base_link">
-    <material>Gazebo/White</material>
-  </gazebo>
   <xacro:define_wheel name_a="front_right" name_b="front_right_joint"  rad="${wheel_radius}" thicc="${wheel_thickness}"  origin_xyz="0.4 -0.3 0.05"/>
   <xacro:define_wheel name_a="front_left" name_b="front_left_joint" rad="${wheel_radius}" thicc="${wheel_thickness}" origin_xyz="0.4 0.3 0.05"/>
   <xacro:define_wheel name_a="back_right" name_b="back_right_joint" rad="${wheel_radius}" thicc="${wheel_thickness}" origin_xyz="-0.4 -0.3 0.05"/>
   <xacro:define_wheel name_a="back_left" name_b="back_left_joint" rad="${wheel_radius}" thicc="${wheel_thickness}" origin_xyz="-0.4 0.3 0.05"/>
+  <gazebo reference="base_link">
+    <material>Gazebo/White</material>
+  </gazebo>
+  <gazebo reference="front_right">
+    <material>Gazebo/Black</material>
+  </gazebo>
+  <gazebo reference="front_left">
+    <material>Gazebo/Black</material>
+  </gazebo>
+<gazebo reference="back_right">
+    <material>Gazebo/Black</material>
+  </gazebo>
+  <gazebo reference="back_left">
+    <material>Gazebo/Black</material>
+  </gazebo>
   <joint name="dummy_joint" type="fixed">
     <origin xyz="0.0 0.0 1" rpy="0.0 0.0 0.0"/>

File: urdf/wheel.xacro (robot description, xacro)
@@ -1,10 +1,11 @@
 <?xml version="1.0"?>
 <robot name="lols"  xmlns:xacro="http://www.ros.org/wiki/xacro">
+    <!-- <xacro:include filename="$(find ohno)/urdf/materials.xacro"/> -->
     <xacro:macro name='define_wheel' params='name_a name_b rad thicc origin_xyz'>
         <link name="${name_a}">
             <inertial>
                 <origin xyz="0 0 0" rpy="0 1.57 1.57"/>
-                <mass value="0.2"/>
-                <inertia ixx="0.0005417" ixy="0" ixz="0" iyy="0.0005417" iyz="0" izz="0.001"/>
+                <mass value="0.5"/>
+                <inertia ixx="0.01" ixy="0" ixz="0" iyy="0.005" iyz="0" izz="0.005"/>
             </inertial>
             <collision>
@@ -18,9 +19,10 @@
                     <cylinder radius="${rad}" length="${thicc}"/>
                 </geometry>
-                <material name="red">
-                    <color rgba="1 0 1 1"/>
-                </material>
+                <material name="red"/>
             </visual>
         </link>
+        <!-- <gazebo reference="${name_a}"> -->
+            <!-- <<material>Gazebo/Black</material> -->
+        <!-- </gazebo> -->
         <joint name="${name_b}" type="continuous">
             <origin xyz="${origin_xyz}" rpy="0 0 0"/>

Commit message: @leander-dsouza, it done.

File: urdf/robo.xacro (robot description, xacro)
@@ -6,13 +6,9 @@
   <xacro:property name="chassis_length" value="1" />
   <xacro:property name="chassis_breadth" value="0.5" />
-  <xacro:property name="chassis_height" value="0.25" />
+  <xacro:property name="chassis_height" value="0.15" />
   <xacro:property name="chassis_mass" value="5" />
   <xacro:include filename="$(find ohno)/urdf/materials.xacro"/>
   <xacro:include filename="$(find ohno)/urdf/wheel.xacro"/>
-  <!-- <xacro:include filename="$(find ohno)/urdf/robo.gazebo"/> -->
-  <gazebo>
-    <static>False</static>
-  </gazebo>
-  <link name="dummy"/>
+  <xacro:include filename="$(find ohno)/urdf/robo.gazebo"/>
   <!-- Base Link -->
   <link name="base_link">
@@ -22,12 +18,12 @@
       <origin xyz="0 0 0.05" rpy="0 0 0" />
       <geometry>
-          <box size="${chassis_length} ${chassis_breadth} ${chassis_height}"/>
+        <box size="${chassis_length} ${chassis_breadth} ${chassis_height}"/>
       </geometry>
     </visual>
     <!-- Base collision, mass and inertia -->
-    <collision>z
-      <origin xyz="0 0 0.05" rpy="0 0 0" />
+    <collision>
+      <origin xyz="0 0 0.05" rpy="0 0 0"/>
       <geometry>
-          <box size="${chassis_length} ${chassis_breadth} ${chassis_height}"/>
+        <box size="${chassis_length} ${chassis_breadth} ${chassis_height}"/>
       </geometry>
     </collision>
@@ -37,27 +33,7 @@
     </inertial>
   </link>
-  <xacro:define_wheel name_a="front_right" name_b="front_right_joint"  rad="${wheel_radius}" thicc="${wheel_thickness}"  origin_xyz="0.4 -0.3 0.05"/>
+  <xacro:define_wheel name_a="front_right" name_b="front_right_joint" rad="${wheel_radius}" thicc="${wheel_thickness}" origin_xyz="0.4 -0.3 0.05"/>
   <xacro:define_wheel name_a="front_left" name_b="front_left_joint" rad="${wheel_radius}" thicc="${wheel_thickness}" origin_xyz="0.4 0.3 0.05"/>
   <xacro:define_wheel name_a="back_right" name_b="back_right_joint" rad="${wheel_radius}" thicc="${wheel_thickness}" origin_xyz="-0.4 -0.3 0.05"/>
   <xacro:define_wheel name_a="back_left" name_b="back_left_joint" rad="${wheel_radius}" thicc="${wheel_thickness}" origin_xyz="-0.4 0.3 0.05"/>
-  <gazebo reference="base_link">
-    <material>Gazebo/White</material>
-  </gazebo>
-  <gazebo reference="front_right">
-    <material>Gazebo/Black</material>
-  </gazebo>
-  <gazebo reference="front_left">
-    <material>Gazebo/Black</material>
-  </gazebo>
-<gazebo reference="back_right">
-    <material>Gazebo/Black</material>
-  </gazebo>
-  <gazebo reference="back_left">
-    <material>Gazebo/Black</material>
-  </gazebo>
-  <joint name="dummy_joint" type="fixed">
-    <origin xyz="0.0 0.0 1" rpy="0.0 0.0 0.0"/>
-    <parent link="dummy"/>
-    <child link="base_link"/>
-  </joint>
 </robot>

File: urdf/wheel.xacro (robot description, xacro)
@@ -1,13 +1,14 @@
 <?xml version="1.0"?>
-<robot name="lols"  xmlns:xacro="http://www.ros.org/wiki/xacro">
+<robot name="lols"
+    xmlns:xacro="http://www.ros.org/wiki/xacro">
     <!-- <xacro:include filename="$(find ohno)/urdf/materials.xacro"/> -->
     <xacro:macro name='define_wheel' params='name_a name_b rad thicc origin_xyz'>
         <link name="${name_a}">
             <inertial>
-                <origin xyz="0 0 0" rpy="0 1.57 1.57"/>
                 <mass value="0.5"/>
                 <inertia ixx="0.01" ixy="0" ixz="0" iyy="0.005" iyz="0" izz="0.005"/>
             </inertial>
             <collision>
+                <origin xyz="0 0 0" rpy="0 1.57 1.57"/>
                 <geometry>
                     <cylinder radius="${rad}" length="${thicc}"/>
@@ -22,7 +23,4 @@
             </visual>
         </link>
-        <!-- <gazebo reference="${name_a}"> -->
-            <!-- <<material>Gazebo/Black</material> -->
-        <!-- </gazebo> -->
         <joint name="${name_b}" type="continuous">
             <origin xyz="${origin_xyz}" rpy="0 0 0"/>

Commit message: fin.

File: urdf/robo.xacro (robot description, xacro)
@@ -6,5 +6,5 @@
   <xacro:property name="chassis_length" value="1" />
   <xacro:property name="chassis_breadth" value="0.5" />
-  <xacro:property name="chassis_height" value="0.15" />
+  <xacro:property name="chassis_height" value="0.25" />
   <xacro:property name="chassis_mass" value="5" />
   <xacro:include filename="$(find ohno)/urdf/materials.xacro"/>
